File: Schematics/Lab-10.brd (EAGLE design)
At the start: 160 x 100 mm, 7 parts, among them Q1 IRLD024

Commit message: Tachometer circuit complete (but messy)
Parts:
- removed R2: 10k, EE445L:RES200MIL
- added C2: (no value), EE445L:CAP100MIL
- added D2: 1N914DO35-7, EE445L:DO35-7
- added IC1: OP350N, EE445L:DIL08
- added R3, R4: (no value), EE445L:RES300MIL
- added R5, R6, R7, R8: (no value), EE445L:RES200MIL
Connections:
- new net N$2: C1.2, D2.C, R3.2
- new net N$3: C2.2, IC1.4, R6.1
- new net N$5: R5.1, R6.2, R7.2
- new net N$6: IC1.3, R7.1, R8.1
- new net TACH_CLIP: IC1.2, R3.1, R4.2
- net GND: now also C2.1, D2.A, IC1.7, R4.1, R5.2
- net TACH: now also IC1.6, R8.2
Changed lines of the file:
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@@
 <layer number="112" name="tSilk" color="7" fill="1" visible="yes" active="yes"/>
 <layer number="113" name="ReferenceLS" color="7" fill="1" visible="no" active="no"/>
+<layer number="114" name="Badge_Outline" color="7" fill="1" visible="yes" active="yes"/>
+<layer number="115" name="ReferenceISLANDS" color="7" fill="1" visible="yes" active="yes"/>
 <layer number="116" name="Patch_BOT" color="9" fill="4" visible="yes" active="yes"/>
 <layer number="117" name="mPads" color="7" fill="1" visible="yes" active="yes"/>
@@
 <attribute name="VALUE" x="-54.2036" y="68.8086" size="0.9906" layer="27" ratio="10"/>
 </element>
-<element name="R2" library="EE445L" package="RES200MIL" value="10k" x="-59.69" y="71.12" smashed="yes">
-<attribute name="NAME" x="-61.6966" y="72.2884" size="0.9906" layer="25" ratio="10"/>
-<attribute name="VALUE" x="-61.8236" y="68.8086" size="0.9906" layer="27" ratio="10"/>
-</element>
 <element name="U$1" library="EE445L" package="TM4C_BOOSTER_PACK" value="TM4C_BP" x="-62.23" y="13.97" smashed="yes"/>
+<element name="D2" library="EE445L" package="DO35-7" value="1N914DO35-7" x="-59.69" y="-3.81" smashed="yes">
+<attribute name="NAME" x="-61.976" y="-2.54" size="1.27" layer="25" ratio="10"/>
+<attribute name="VALUE" x="-61.976" y="-6.477" size="1.27" layer="27" ratio="10"/>
+</element>
+<element name="R3" library="EE445L" package="RES300MIL" value="" x="-59.69" y="-10.16" smashed="yes">
+<attribute name="NAME" x="-62.23" y="-8.8646" size="0.9906" layer="25" ratio="10"/>
+<attribute name="VALUE" x="-61.3156" y="-10.6426" size="0.9906" layer="27" ratio="10"/>
+</element>
+<element name="R4" library="EE445L" package="RES300MIL" value="" x="-59.69" y="-15.24" smashed="yes">
+<attribute name="NAME" x="-62.23" y="-13.9446" size="0.9906" layer="25" ratio="10"/>
+<attribute name="VALUE" x="-61.3156" y="-15.7226" size="0.9906" layer="27" ratio="10"/>
+</element>
+<element name="IC1" library="EE445L" package="DIL08" value="OP350N" x="-57.15" y="-21.59" smashed="yes">
+<attribute name="MF" value="" x="-57.15" y="-21.59" size="1.778" layer="27" display="off"/>
+<attribute name="MPN" value="AD8031BNZ" x="-57.15" y="-21.59" size="1.778" layer="27" display="off"/>
+<attribute name="NAME" x="-62.484" y="-24.511" size="1.27" layer="25" ratio="10" rot="R90"/>
+<attribute name="OC_FARNELL" value="1438575" x="-57.15" y="-21.59" size="1.778" layer="27" display="off"/>
+<attribute name="OC_NEWARK" value="15P0920" x="-57.15" y="-21.59" size="1.778" layer="27" display="off"/>
+<attribute name="VALUE" x="-60.706" y="-22.225" size="1.27" layer="27" ratio="10"/>
+</element>
+<element name="R5" library="EE445L" package="RES200MIL" value="" x="-60.96" y="-29.21" smashed="yes">
+<attribute name="NAME" x="-62.9666" y="-28.0416" size="0.9906" layer="25" ratio="10"/>
+<attribute name="VALUE" x="-63.0936" y="-31.5214" size="0.9906" layer="27" ratio="10"/>
+</element>
+<element name="R6" library="EE445L" package="RES200MIL" value="" x="-60.96" y="-33.02" smashed="yes">
+<attribute name="NAME" x="-62.9666" y="-31.8516" size="0.9906" layer="25" ratio="10"/>
+<attribute name="VALUE" x="-63.0936" y="-35.3314" size="0.9906" layer="27" ratio="10"/>
+</element>
+<element name="R7" library="EE445L" package="RES200MIL" value="" x="-60.96" y="-36.83" smashed="yes">
+<attribute name="NAME" x="-62.9666" y="-35.6616" size="0.9906" layer="25" ratio="10"/>
+<attribute name="VALUE" x="-63.0936" y="-39.1414" size="0.9906" layer="27" ratio="10"/>
+</element>
+<element name="R8" library="EE445L" package="RES200MIL" value="" x="-60.96" y="-40.64" smashed="yes">
+<attribute name="NAME" x="-62.9666" y="-39.4716" size="0.9906" layer="25" ratio="10"/>
+<attribute name="VALUE" x="-63.0936" y="-42.9514" size="0.9906" layer="27" ratio="10"/>
+</element>
+<element name="C2" library="EE445L" package="CAP100MIL" value="" x="-62.23" y="-45.72" smashed="yes">
+<attribute name="NAME" x="-64.008" y="-44.323" size="1.27" layer="25" ratio="10"/>
+<attribute name="VALUE" x="-64.008" y="-48.387" size="1.27" layer="27" ratio="10"/>
+</element>
 </elements>
 <signals>
@@
 <contactref element="JP1" pad="6"/>
 <contactref element="Q1" pad="P$4"/>
-<wire x1="-16.51" y1="73.66" x2="-15.24" y2="77.47" width="0" layer="19" extent="1-1"/>
+<contactref element="D2" pad="A"/>
+<contactref element="R4" pad="1"/>
+<contactref element="IC1" pad="7"/>
+<contactref element="C2" pad="1"/>
+<contactref element="R5" pad="2"/>
+<wire x1="-58.42" y1="-29.21" x2="-63.5" y2="-45.72" width="0" layer="19" extent="1-1"/>
+<wire x1="-58.42" y1="-17.78" x2="-58.42" y2="-29.21" width="0" layer="19" extent="1-1"/>
+<wire x1="-63.5" y1="-15.24" x2="-58.42" y2="-17.78" width="0" layer="19" extent="1-1"/>
+<wire x1="-55.88" y1="-3.81" x2="-63.5" y2="-15.24" width="0" layer="19" extent="1-1"/>
+<wire x1="-16.51" y1="73.66" x2="-55.88" y2="-3.81" width="0" layer="19" extent="1-1"/>
+<wire x1="-15.24" y1="77.47" x2="-16.51" y2="73.66" width="0" layer="19" extent="1-1"/>
 </signal>
 <signal name="+3V3">
@@
 <signal name="TACH">
 <contactref element="U$1" pad="J1-7"/>
+<contactref element="IC1" pad="6"/>
+<contactref element="R8" pad="2"/>
+<wire x1="-55.88" y1="-17.78" x2="-58.42" y2="-40.64" width="0" layer="19" extent="1-1"/>
+<wire x1="-62.23" y1="21.59" x2="-55.88" y2="-17.78" width="0" layer="19" extent="1-1"/>
 </signal>
 <signal name="N$1">
@@
 <wire x1="-46.99" y1="71.12" x2="-27.94" y2="77.47" width="0" layer="19" extent="1-1"/>
 </signal>
+<signal name="N$2">
+<contactref element="D2" pad="C"/>
+<contactref element="C1" pad="2"/>
+<contactref element="R3" pad="2"/>
+<wire x1="-55.88" y1="-10.16" x2="-63.5" y2="-3.81" width="0" layer="19" extent="1-1"/>
+<wire x1="-29.21" y1="71.12" x2="-63.5" y2="-3.81" width="0" layer="19" extent="1-1"/>
+</signal>
+<signal name="TACH_CLIP">
+<contactref element="R3" pad="1"/>
+<contactref element="R4" pad="2"/>
+<contactref element="IC1" pad="2"/>
+<wire x1="-55.88" y1="-15.24" x2="-58.42" y2="-25.4" width="0" layer="19" extent="1-1"/>
+<wire x1="-63.5" y1="-10.16" x2="-55.88" y2="-15.24" width="0" layer="19" extent="1-1"/>
+</signal>
+<signal name="N$3">
+<contactref element="IC1" pad="4"/>
+<contactref element="C2" pad="2"/>
+<contactref element="R6" pad="1"/>
+<wire x1="-63.5" y1="-33.02" x2="-60.96" y2="-45.72" width="0" layer="19" extent="1-1"/>
+<wire x1="-53.34" y1="-25.4" x2="-63.5" y2="-33.02" width="0" layer="19" extent="1-1"/>
+</signal>
+<signal name="N$5">
+<contactref element="R6" pad="2"/>
+<contactref element="R5" pad="1"/>
+<contactref element="R7" pad="2"/>
+<wire x1="-58.42" y1="-33.02" x2="-58.42" y2="-36.83" width="0" layer="19" extent="1-1"/>
+<wire x1="-63.5" y1="-29.21" x2="-58.42" y2="-33.02" width="0" layer="19" extent="1-1"/>
+</signal>
+<signal name="N$6">
+<contactref element="R7" pad="1"/>
+<contactref element="R8" pad="1"/>
+<contactref element="IC1" pad="3"/>
+<wire x1="-63.5" y1="-36.83" x2="-63.5" y2="-40.64" width="0" layer="19" extent="1-1"/>
+<wire x1="-55.88" y1="-25.4" x2="-63.5" y2="-36.83" width="0" layer="19" extent="1-1"/>
+</signal>
 </signals>
